File: mounting holes.kicad_sch (KiCad schematic)
At the start: 0 parts

Commit message: analog schematics added
some questions
Parts:
- added H1, H10, H11, H12, H13, H14, H15, H16, H17, H18, H19, H2, H20, H21, H22, H23, H24, H25, H26, H3, H4, H5, H6, H7, H8, H9: MountingHole, cipulot_parts:HOLE_M2, symbol Mechanical:MountingHole

Commit message: component placement
Parts:
- removed H1, H10, H11, H12, H13, H14, H15, H16, H17, H18, H19, H2, H20, H21, H22, H23, H24, H25, H26, H3, H4, H5, H6, H7, H8, H9: MountingHole, cipulot_parts:HOLE_M2, symbol Mechanical:MountingHole

Commit message: created simplified version
Parts:
- added H1, H10, H11, H12, H13, H14, H15, H16, H17, H2, H3, H4, H5, H6, H7, H8, H9: MountingHole, cipulot_parts:HOLE_M2, symbol Mechanical:MountingHole
