File: travaulta simplified.kicad_pcb (KiCad board)
At the start: 4 copper layers, 209.7 x 76.4 mm, 101 parts, among them SW1 EC_SW, SW10 EC_SW, SW11 EC_SW, SW12 EC_SW, SW13 EC_SW, SW14 EC_SW, SW15 EC_SW, SW16 EC_SW, SW17 EC_SW, SW18 EC_SW, SW19 EC_SW, SW2 EC_SW, SW20 EC_SW, SW21 EC_SW, SW22 EC_SW, SW23 EC_SW, SW24 EC_SW, SW25 EC_SW, SW26 EC_SW, SW27 EC_SW, SW28 EC_SW, SW29 EC_SW, SW3 EC_SW, SW30 EC_SW, SW31 EC_SW, SW32 EC_SW, SW33 EC_SW, SW34 EC_SW, SW35 EC_SW, SW36 EC_SW, SW37 EC_SW, SW38 BOOT0, SW4 EC_SW, SW5 EC_SW, SW6 EC_SW, SW7 EC_SW, SW8 EC_SW, SW9 EC_SW, U1 STM32F411CCUx, U2 XC6206PxxxMR, U3 74HC4051, U4 74HC4051, U5 OPA350, Y1 16 MHz

Commit message: cleaned pcb, silkscreen, created first plates
Parts:
- moved R20 12.4 mm to (193.7, 101.6)
- moved JP1 10.4 mm to (137.9, 120.7), turned to 45 degrees
- moved R12 6.60 mm to (157.2, 101.6)
- moved R21 6.35 mm to (140.0, 120.4), turned to -90 degrees
- moved SW38 3.49 mm to (181.0, 113.0)
- moved C14 3.45 mm to (140.7, 114.9), turned to 180 degrees
- moved C15 2.53 mm to (149.0, 118.0)
- moved R23 2.06 mm to (139.6, 118.5), turned to 180 degrees
- moved R1 1.26 mm to (148.5, 106.4)
- moved R2 1.26 mm to (151.5, 106.4)
- moved R4 1.26 mm to (153.0, 105.9)
- moved R8 1.26 mm to (150.5, 106.4)
- moved R9 1.26 mm to (149.5, 106.4)
- moved R6 1.22 mm to (150.7, 119.5)
- moved Y1 1.22 mm to (154.6, 118.7)
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Connections:
- R1 pad 2: ROW0 -> ROW3
- R2 pad 1: ROW3 -> ROW2
- R8 pad 1: ROW2 -> ROW1
- R9 pad 2: ROW1 -> ROW0
- U1 pad 14: unconnected-(U1-PA4-Pad14) -> APLEX_OUT_PIN_0
- U1 pad 18: APLEX_OUT_PIN_0 -> APLEX_EN_PIN_0
- U1 pad 19: unconnected-(U1-PB1-Pad19) -> APLEX_EN_PIN_1
- U1 pad 42: APLEX_EN_PIN_1 -> unconnected-(U1-PB6-Pad42)
- U1 pad 43: APLEX_EN_PIN_0 -> unconnected-(U1-PB7-Pad43)
Routing:
- net AMUX_SEL_2: track 0.00 -> 152.6 mm, vias 0 -> 2
- net AMUX_SEL_1: track 0.00 -> 150.7 mm, vias 0 -> 2
- net AMUX_SEL_0: track 0.00 -> 149.0 mm, vias 0 -> 2
- net APLEX_OUT_PIN_0: track 5.64 -> 138.0 mm, vias 0 -> 5
- net APLEX_EN_PIN_1: track 0.00 -> 73.7 mm, vias 0 -> 4
- net APLEX_EN_PIN_0: track 0.00 -> 60.2 mm
- net COL5: track 67.8 -> 125.9 mm
- net ROW0: track 320.1 -> 373.4 mm, vias 11 -> 13
- net COL6: track 55.3 -> 91.5 mm, vias 3 -> 5
- net ROW1: track 313.8 -> 348.8 mm, vias 10 -> 12
- net BOOT0: track 2.47 -> 37.1 mm, vias 1 -> 0
- net VBAT: track 262.7 -> 296.7 mm
- net COL9: track 101.8 -> 129.8 mm
- net COL7: track 80.4 -> 104.2 mm, vias 4 -> 6
- net ROW3: track 201.2 -> 220.8 mm, vias 6 -> 8
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Other:
- board text added: "Travaulta v1.0"
- board text added: "changed u3 and u4 to smd, instead of through hole, is that okay?"
- board text added: "designed by Calvin#0563 based on projectcain#5265's vault35"
- board text removed: "design by Calvin#0563 based on the vault35 by projectcain#5265"
- board text removed: "housing edge cut interference???"
- board text removed: "something not working with the footprint, no power 3v3 at switch"
- board text removed: "travaulta (topre-vault[a]35)"

Commit message: created more plates
Connections:
- U4 pad 5: unconnected-(U4-A5-Pad5) -> GND
Changed lines of the file:
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@@
   (net 55 "unconnected-(U1-PB8-Pad45)")
   (net 56 "unconnected-(U1-PB9-Pad46)")
-  (net 57 "unconnected-(U4-A5-Pad5)")
-  (net 58 "unconnected-(USB1-SBU2-Pad3)")
-  (net 59 "unconnected-(USB1-SBU1-Pad9)")
-  (net 60 "unconnected-(U1-PA5-Pad15)")
-  (net 61 "unconnected-(U1-PA6-Pad16)")
-  (net 62 "unconnected-(U1-PA7-Pad17)")
-  (net 63 "unconnected-(U1-PB7-Pad43)")
+  (net 57 "unconnected-(USB1-SBU2-Pad3)")
+  (net 58 "unconnected-(USB1-SBU1-Pad9)")
+  (net 59 "unconnected-(U1-PA5-Pad15)")
+  (net 60 "unconnected-(U1-PA6-Pad16)")
+  (net 61 "unconnected-(U1-PA7-Pad17)")
+  (net 62 "unconnected-(U1-PB7-Pad43)")
   (footprint "cipulot_parts:ecs_pad_1U_no_ring" locked (layer "F.Cu")
     (at 211.1375 76.2)
@@
       (net 8 "APLEX_OUT_PIN_0") (pinfunction "PA4") (pintype "bidirectional"))
     (pad "15" smd roundrect (at -1.75 -3.4375 90) (size 0.25 0.875) (layers "B.Cu" "B.Paste" "B.Mask") (roundrect_rratio 0.25)
-      (net 60 "unconnected-(U1-PA5-Pad15)") (pinfunction "PA5") (pintype "bidirectional"))
+      (net 59 "unconnected-(U1-PA5-Pad15)") (pinfunction "PA5") (pintype "bidirectional"))
     (pad "16" smd roundrect (at -1.25 -3.4375 90) (size 0.25 0.875) (layers "B.Cu" "B.Paste" "B.Mask") (roundrect_rratio 0.25)
-      (net 61 "unconnected-(U1-PA6-Pad16)") (pinfunction "PA6") (pintype "bidirectional"))
+      (net 60 "unconnected-(U1-PA6-Pad16)") (pinfunction "PA6") (pintype "bidirectional"))
     (pad "17" smd roundrect (at -0.75 -3.4375 90) (size 0.25 0.875) (layers "B.Cu" "B.Paste" "B.Mask") (roundrect_rratio 0.25)
-      (net 62 "unconnected-(U1-PA7-Pad17)") (pinfunction "PA7") (pintype "bidirectional"))
+      (net 61 "unconnected-(U1-PA7-Pad17)") (pinfunction "PA7") (pintype "bidirectional"))
     (pad "18" smd roundrect (at -0.25 -3.4375 90) (size 0.25 0.875) (layers "B.Cu" "B.Paste" "B.Mask") (roundrect_rratio 0.25)
       (net 48 "APLEX_EN_PIN_0") (pinfunction "PB0") (pintype "bidirectional"))
@@
       (net 50 "unconnected-(U1-PB6-Pad42)") (pinfunction "PB6") (pintype "bidirectional"))
     (pad "43" smd roundrect (at -0.25 3.4375 90) (size 0.25 0.875) (layers "B.Cu" "B.Paste" "B.Mask") (roundrect_rratio 0.25)
-      (net 63 "unconnected-(U1-PB7-Pad43)") (pinfunction "PB7") (pintype "bidirectional"))
+      (net 62 "unconnected-(U1-PB7-Pad43)") (pinfunction "PB7") (pintype "bidirectional"))
     (pad "44" smd roundrect (at -0.75 3.4375 90) (size 0.25 0.875) (layers "B.Cu" "B.Paste" "B.Mask") (roundrect_rratio 0.25)
       (net 46 "BOOT0") (pinfunction "BOOT0") (pintype "input"))
@@
       (net 1 "GND") (pinfunction "A7") (pintype "passive"))
     (pad "5" smd rect (at 0.32258 -2.97434 90) (size 0.4191 1.778) (layers "B.Cu" "B.Paste" "B.Mask")
-      (net 57 "unconnected-(U4-A5-Pad5)") (pinfunction "A5") (pintype "passive"))
+      (net 1 "GND") (pinfunction "A5") (pintype "passive"))
     (pad "6" smd rect (at 0.97282 -2.97434 90) (size 0.4191 1.778) (layers "B.Cu" "B.Paste" "B.Mask")
       (net 48 "APLEX_EN_PIN_0") (pinfunction "~{E}") (pintype "input"))
@@
       (net 4 "VCC") (pinfunction "VBUS") (pintype "input"))
     (pad "3" smd rect (at -1.75 7.65) (size 0.3 1.3) (layers "B.Cu" "B.Paste" "B.Mask")
-      (net 58 "unconnected-(USB1-SBU2-Pad3)") (pinfunction "SBU2") (pintype "input+no_connect"))
+      (net 57 "unconnected-(USB1-SBU2-Pad3)") (pinfunction "SBU2") (pintype "input+no_connect"))
     (pad "4" smd rect (at -1.25 7.65) (size 0.3 1.3) (layers "B.Cu" "B.Paste" "B.Mask")
       (net 33 "Net-(USB1-CC1)") (pinfunction "CC1") (pintype "input"))
@@
       (net 3 "D+") (pinfunction "DP2") (pintype "input"))
     (pad "9" smd rect (at 1.25 7.65) (size 0.3 1.3) (layers "B.Cu" "B.Paste" "B.Mask")
-      (net 59 "unconnected-(USB1-SBU1-Pad9)") (pinfunction "SBU1") (pintype "input+no_connect"))
+      (net 58 "unconnected-(USB1-SBU1-Pad9)") (pinfunction "SBU1") (pintype "input+no_connect"))
     (pad "10" smd rect (at 1.75 7.65) (size 0.3 1.3) (layers "B.Cu" "B.Paste" "B.Mask")
       (net 34 "Net-(USB1-CC2)") (pinfunction "CC2") (pintype "input"))
