File: travaulta rgb.kicad_pcb (KiCad board)
At the start: 4 copper layers, 209.7 x 76.4 mm, 113 parts, among them SW1 EC_SW, SW10 EC_SW, SW11 EC_SW, SW12 EC_SW, SW13 EC_SW, SW14 EC_SW, SW15 EC_SW, SW16 EC_SW, SW17 EC_SW, SW18 EC_SW, SW19 EC_SW, SW2 EC_SW, SW20 EC_SW, SW21 EC_SW, SW22 EC_SW, SW23 EC_SW, SW24 EC_SW, SW25 EC_SW, SW26 EC_SW, SW27 EC_SW, SW28 EC_SW, SW29 EC_SW, SW3 EC_SW, SW30 EC_SW, SW31 EC_SW, SW32 EC_SW, SW33 EC_SW, SW34 EC_SW, SW35 EC_SW, SW36 EC_SW, SW37 EC_SW, SW38 BOOT0, SW4 EC_SW, SW5 EC_SW, SW6 EC_SW, SW7 EC_SW, SW8 EC_SW, SW9 EC_SW, U1 STM32F411CCUx, U2 XC6206PxxxMR, U3 74HC4051, U4 74HC4051, U5 OPA350, Y1 16 MHz

Commit message: first rough rgb version done
no idea about interferences and all.
Parts:
- added U6: SN74AHCT1G125, Package_TO_SOT_SMD:SOT-23-5, B.Cu at (68.3, 73.0)
- moved LED4 1.21 mm to (228.5, 69.5)
- moved LED2 0.12 mm to (125.3, 69.6)
Connections:
- LED1 pad 4: rgb underglow -> underglow_5V
- U1 pad 17: unconnected-(U1-PA7-Pad17) -> underglow_3V3
Routing:
- net +5V: track 3.42 -> 330.7 mm, vias 0 -> 9
- net underglow_3V3: track 0.00 -> 111.2 mm, vias 0 -> 2
- net Net-(LED1-DOUT): track 0.00 -> 61.5 mm
- net Net-(LED2-DOUT): track 0.00 -> 60.9 mm, vias 0 -> 2
- net Net-(LED6-DOUT): track 0.00 -> 56.2 mm, vias 0 -> 2
- net Net-(LED7-DOUT): track 0.00 -> 55.8 mm
- net Net-(LED3-DOUT): track 0.00 -> 50.9 mm
- net Net-(LED5-DOUT): track 0.00 -> 46.3 mm
- net Net-(LED4-DOUT): track 0.00 -> 22.8 mm
- net underglow_5V: track 0.00 -> 2.63 mm
- net GND: track 26.0 -> 28.4 mm, vias 274 -> 275
- net D-: track 128.7 -> 127.8 mm
- net D+: track 128.6 -> 128.0 mm
