File: travaulta rgb.kicad_sch (KiCad schematic)
At the start: 34 parts, among them SW38 BOOT0, U1 STM32F411CCUx, U2 XC6206PxxxMR, Y1 16 MHz

Commit message: first rough rgb version done
no idea about interferences and all.
Parts:
- added U6: SN74AHCT1G125, Package_TO_SOT_SMD:SOT-23-5, symbol cipulot_parts:SN74AHCT1G125
Connections:
- net +5V: now also U6.5 (VCC)
- net GND: now also U6.1 (~{OE}), U6.3 (GND)
- net underglow_3V3: now reaches U1.17 (PA7)
- net underglow_3V3: now also U6.2 (A)
- net rgb underglow renamed underglow_5V
- net underglow_5V: now also U6.4 (B)
- no-connect marks 18 -> 17
Other:
- note added: "LED Logic Level Shifter"
Changed lines of the file:
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@@
   (junction (at 169.545 173.99) (diameter 0) (color 0 0 0 0)
+  )
+  (junction (at 147.32 83.82) (diameter 0) (color 0 0 0 0)
   )
   (junction (at 66.675 99.695) (diameter 0) (color 0 0 0 0)
@@
   (no_connect (at 48.895 79.375))
   (no_connect (at 81.915 79.375))
-  (no_connect (at 81.915 74.295))
   (no_connect (at 48.895 81.915))
   (no_connect (at 81.915 69.215))
@@
     (stroke (width 0) (type default))
   )
+  (wire (pts (xy 137.16 83.82) (xy 147.32 83.82))
+    (stroke (width 0) (type default))
+  )
   (wire (pts (xy 81.915 92.075) (xy 94.615 92.075))
     (stroke (width 0) (type default))
@@
     (stroke (width 0) (type default))
   )
+  (wire (pts (xy 147.32 83.82) (xy 147.32 83.185))
+    (stroke (width 0) (type default))
+  )
   (wire (pts (xy 169.545 175.26) (xy 169.545 173.99))
     (stroke (width 0) (type default))
@@
     (stroke (width 0) (type default))
   )
+  (wire (pts (xy 147.32 84.455) (xy 147.32 83.82))
+    (stroke (width 0) (type default))
+  )
   (wire (pts (xy 66.675 99.695) (xy 69.215 99.695))
     (stroke (width 0) (type default))
   )
   (wire (pts (xy 24.13 92.075) (xy 26.67 92.075))
+    (stroke (width 0) (type default))
+  )
+  (wire (pts (xy 137.16 78.105) (xy 137.16 83.82))
     (stroke (width 0) (type default))
   )
@@
   )
   (text "Reset Pullup" (at 160.655 123.825 0)
+    (effects (font (size 1.27 1.27)) (justify left bottom))
+  )
+  (text "LED Logic Level Shifter" (at 126.365 58.42 0)
     (effects (font (size 1.27 1.27)) (justify left bottom))
   )
@@
     )
   )
+  (global_label "underglow_3V3" (shape input) (at 137.16 73.025 180) (fields_autoplaced)
+    (effects (font (size 1.27 1.27)) (justify right))
+    (property "Intersheetrefs" "${INTERSHEET_REFS}" (at 120.1635 73.025 0)
+      (effects (font (size 1.27 1.27)) (justify right) hide)
+    )
+  )
   (global_label "ROW2" (shape input) (at 24.13 94.615 180) (fields_autoplaced)
     (effects (font (size 1.27 1.27)) (justify right))
@@
     )
   )
+  (global_label "underglow_5V" (shape input) (at 126.365 39.37 180) (fields_autoplaced)
+    (effects (font (size 1.27 1.27)) (justify right))
+    (property "Intersheetrefs" "${INTERSHEET_REFS}" (at 110.578 39.37 0)
+      (effects (font (size 1.27 1.27)) (justify right) hide)
+    )
+  )
   (global_label "XTAL0" (shape input) (at 48.895 41.275 180) (fields_autoplaced)
     (effects (font (size 1.27 1.27)) (justify right))
@@
     )
   )
-  (global_label "rgb underglow" (shape input) (at 93.345 48.26 0) (fields_autoplaced)
-    (effects (font (size 1.27 1.27)) (justify left))
-    (property "Intersheetrefs" "${INTERSHEET_REFS}" (at 109.7125 48.26 0)
-      (effects (font (size 1.27 1.27)) (justify left) hide)
-    )
-  )
-  (global_label "rgb underglow" (shape input) (at 126.365 39.37 180) (fields_autoplaced)
-    (effects (font (size 1.27 1.27)) (justify right))
-    (property "Intersheetrefs" "${INTERSHEET_REFS}" (at 110.2843 39.2906 0)
-      (effects (font (size 1.27 1.27)) (justify right) hide)
-    )
-  )
   (global_label "D-" (shape input) (at 45.085 182.245 0) (fields_autoplaced)
     (effects (font (size 1.27 1.27)) (justify left))
@@
     )
   )
+  (global_label "underglow_5V" (shape output) (at 157.48 73.025 0) (fields_autoplaced)
+    (effects (font (size 1.27 1.27)) (justify left))
+    (property "Intersheetrefs" "${INTERSHEET_REFS}" (at 173.267 73.025 0)
+      (effects (font (size 1.27 1.27)) (justify left) hide)
+    )
+  )
   (global_label "AMUX_SEL_0" (shape output) (at 48.895 71.755 180) (fields_autoplaced)
     (effects (font (size 1.27 1.27)) (justify right))
@@
     )
   )
+  (global_label "underglow_3V3" (shape input) (at 81.915 74.295 0) (fields_autoplaced)
+    (effects (font (size 1.27 1.27)) (justify left))
+    (property "Intersheetrefs" "${INTERSHEET_REFS}" (at 98.9115 74.295 0)
+      (effects (font (size 1.27 1.27)) (justify left) hide)
+    )
+  )
   (global_label "D-" (shape input) (at 39.37 131.445 0) (fields_autoplaced)
     (effects (font (size 1.27 1.27)) (justify left))
@@
     )
   )
+  (symbol (lib_id "cipulot_parts:SN74AHCT1G125") (at 147.32 75.565 0) (unit 1)
+    (in_bom yes) (on_board yes) (dnp no)
+    (property "Reference" "U6" (at 156.845 60.9631 0)
+      (effects (font (size 1.27 1.27)))
+    )
+    (property "Value" "SN74AHCT1G125" (at 156.845 63.5 0)
+      (effects (font (size 1.27 1.27)))
+    )
+    (property "Footprint" "Package_TO_SOT_SMD:SOT-23-5" (at 148.59 89.535 0)
+      (effects (font (size 1.27 1.27)) hide)
+    )
+    (property "Datasheet" "https://www.ti.com/cn/lit/ds/symlink/sn74ahct1g125.pdf?ts=1660138492922" (at 124.46 89.535 0)
+      (effects (font (size 1.27 1.27)) hide)
+    )
+    (property "LCSC" "C7484" (at 147.32 75.565 0)
+      (effects (font (size 1.27 1.27)) hide)
+    )
+    (pin "1")
+    (pin "2")
+    (pin "3")
+    (pin "4")
+    (pin "5")
+    (instances
+      (project "travaulta rgb"
+        (path "/690df46b-b605-4617-b545-6aaced86d0fc"
+          (reference "U6") (unit 1)
+        )
+      )
+    )
+  )
   (symbol (lib_id "power:+3V3") (at 167.005 131.445 0) (unit 1)
     (in_bom yes) (on_board yes) (dnp no) (fields_autoplaced)
@@
         (path "/690df46b-b605-4617-b545-6aaced86d0fc"
           (reference "#PWR0151") (unit 1)
+        )
+      )
+    )
+  )
+  (symbol (lib_id "power:GND") (at 147.32 84.455 0) (unit 1)
+    (in_bom yes) (on_board yes) (dnp no)
+    (property "Reference" "#PWR05" (at 147.32 90.805 0)
+      (effects (font (size 1.27 1.27)) hide)
+    )
+    (property "Value" "GND" (at 149.86 88.265 0)
+      (effects (font (size 1.27 1.27)) (justify right))
+    )
+    (property "Footprint" "" (at 147.32 84.455 0)
+      (effects (font (size 1.27 1.27)) hide)
+    )
+    (property "Datasheet" "" (at 147.32 84.455 0)
+      (effects (font (size 1.27 1.27)) hide)
+    )
+    (pin "1")
+    (instances
+      (project "travaulta rgb"
+        (path "/690df46b-b605-4617-b545-6aaced86d0fc"
+          (reference "#PWR05") (unit 1)
         )
       )
@@
         )
       )
+    )
+  )
+  (symbol (lib_id "power:+5V") (at 147.32 62.865 0) (unit 1)
+    (in_bom yes) (on_board yes) (dnp no) (fields_autoplaced)
+    (property "Reference" "#PWR04" (at 147.32 66.675 0)
+      (effects (font (size 1.27 1.27)) hide)
+    )
+    (property "Value" "+5V" (at 147.32 59.2605 0)
+      (effects (font (size 1.27 1.27)))
+    )
+    (property "Footprint" "" (at 147.32 62.865 0)
+      (effects (font (size 1.27 1.27)) hide)
+    )
+    (property "Datasheet" "" (at 147.32 62.865 0)
+      (effects (font (size 1.27 1.27)) hide)
+    )
+    (pin "1")
+    (instances
+      (project "travaulta rgb"
+        (path "/690df46b-b605-4617-b545-6aaced86d0fc"
+          (reference "#PWR04") (unit 1)
+        )
+      )
