File: travaulta revision.kicad_pcb (KiCad board)
At the start: 4 copper layers, 209.7 x 76.4 mm, 106 parts, among them SW1 EC_SW, SW10 EC_SW, SW11 EC_SW, SW12 EC_SW, SW13 EC_SW, SW14 EC_SW, SW15 EC_SW, SW16 EC_SW, SW17 EC_SW, SW18 EC_SW, SW19 EC_SW, SW2 EC_SW, SW20 EC_SW, SW21 EC_SW, SW22 EC_SW, SW23 EC_SW, SW24 EC_SW, SW25 EC_SW, SW26 EC_SW, SW27 EC_SW, SW28 EC_SW, SW29 EC_SW, SW3 EC_SW, SW30 EC_SW, SW31 EC_SW, SW32 EC_SW, SW33 EC_SW, SW34 EC_SW, SW35 EC_SW, SW36 EC_SW, SW37 EC_SW, SW38 BOOT0, SW4 EC_SW, SW5 EC_SW, SW6 EC_SW, SW7 EC_SW, SW8 EC_SW, SW9 EC_SW, U1 STM32F401CBUx, U2 XC6206PxxxMR, U3 74HC4051, U4 74HC4051, U5 OPA350, Y1 8 MHz

Commit message: revision routing
Parts:
- moved R21 6.84 mm to (146.8, 119.4), turned to 0 degrees
- moved JP1 6.82 mm to (144.5, 120.7), turned to 180 degrees
- moved R13 4.18 mm to (75.8, 107.2), turned to 180 degrees
- moved R23 2.63 mm to (142.1, 119.4)
- moved C14 2.22 mm to (140.7, 112.7)
- moved U5 2.15 mm to (144.4, 116.2)
- moved C13 1.75 mm to (88.9, 104.5), turned to 180 degrees
- moved U3 0.79 mm to (205.6, 108.0)
- moved U4 0.79 mm to (92.9, 108.0)
Connections:
- U3 pad 4: GND -> APLEX_EN_PIN_1
Routing:
- net COL10: track 140.3 -> 89.1 mm, vias 4 -> 2
- net GND: track 87.7 -> 37.7 mm, vias 167 -> 149
- net APLEX_EN_PIN_1: track 22.5 -> 72.4 mm, vias 1 -> 4
- net COL9: track 84.1 -> 131.6 mm, vias 3 -> 5
- net VBAT: track 299.2 -> 271.9 mm, vias 7 -> 9
- net COL8: track 84.1 -> 73.1 mm
- net COL6: track 98.7 -> 87.8 mm
- net AMUX_SEL_0: track 155.8 -> 146.1 mm, vias 1 -> 2
- net COL1: track 86.3 -> 91.3 mm
- net Net-(JP1-B): track 5.00 -> 8.98 mm
- net APLEX_OUT_PIN_0: track 87.0 -> 83.6 mm, vias 2 -> 3
- net ADC: track 15.4 -> 12.5 mm
- net COL0: track 76.8 -> 79.3 mm
- net COL3: track 112.5 -> 115.0 mm
- net AMUX_SEL_1: track 151.4 -> 149.4 mm, vias 1 -> 2
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- added copper zone on F.Cu, net GND

Commit message: rerouting in progress
Parts:
- moved C12 1.84 mm to (203.1, 104.5)
- moved R14 1.11 mm to (208.5, 112.1)
- moved R5 0.10 mm to (222.7, 107.2), turned to 0 degrees
Connections:
- U3 pad 4: APLEX_EN_PIN_1 -> GND
Routing:
- net APLEX_OUT_PIN_0: track 83.6 -> 142.5 mm, vias 3 -> 6
- net VBAT: track 271.9 -> 319.3 mm
- net COL9: track 131.6 -> 85.5 mm, vias 5 -> 3
- net COL8: track 73.1 -> 82.7 mm
- net APLEX_EN_PIN_1: track 72.4 -> 78.0 mm, vias 4 -> 2
- net COL7: track 96.9 -> 101.7 mm, vias 4 -> 6
- net COL6: track 87.8 -> 92.3 mm, vias 3 -> 5
- net AMUX_SEL_2: track 151.7 -> 149.0 mm
- net COL5: track 126.5 -> 129.2 mm
- net AMUX_SEL_1: track 149.4 -> 152.1 mm
- net AMUX_SEL_0: track 146.1 -> 147.3 mm
- net VCC: track 14.9 -> 14.0 mm
- net COL10: track 89.1 -> 89.9 mm
- net GND: vias 149 -> 161
Other:
- board text added: "align height of routing, make cleaner more unform"

Commit message: tiny rerouting
Parts:
- moved R16 0.13 mm to (228.6, 101.6)
Routing:
- net ROW3: vias 9 -> 8
Other:
- board text added: "ADD NEW FRESH GND VIAS"
- board text removed: "GND in inner layers usb shield layer outside?"
Changed lines of the file:
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@@
   )
   (footprint "Resistor_SMD:R_0402_1005Metric" (layer "B.Cu")
-    (at 228.6 101.473 90)
+    (at 228.6 101.6 90)
     (descr "Resistor SMD 0402 (1005 Metric), square (rectangular) end terminal, IPC_7351 nominal, (Body size source: IPC-SM-782 page 72, https://www.pcb-3d.com/wordpress/wp-content/uploads/ipc-sm-782a_amendment_1_and_2.pdf), generated with kicad-footprint-generator")
     (tags "resistor")
@@
   (gr_arc locked (start 249.184374 102.433999) (mid 249.931233 100.630857) (end 251.734375 99.884)
     (stroke (width 0.05) (type solid)) (layer "Edge.Cuts"))
-  (gr_text "GND in inner layers\nusb shield layer outside?\n" (at 73.81875 142.875) (layer "B.Cu")
+  (gr_text "ADD NEW FRESH GND VIAS" (at 70.64375 136.525) (layer "B.Cu")
     (effects (font (size 1.5 1.5) (thickness 0.3) bold) (justify left bottom))
   )
@@
   (segment (start 140.1725 114.230655) (end 140.1725 112.7125) (width 0.25) (layer "B.Cu") (net 8))
   (segment (start 145.914195 85.725) (end 145.669 85.479805) (width 0.25) (layer "F.Cu") (net 9))
+  (segment (start 146.133201 85.944006) (end 145.914195 85.725) (width 0.25) (layer "F.Cu") (net 9))
+  (segment (start 151.8125 86.345453) (end 151.411053 85.944006) (width 0.25) (layer "F.Cu") (net 9))
+  (segment (start 151.8125 99.765195) (end 151.8125 86.51875) (width 0.25) (layer "F.Cu") (net 9))
   (segment (start 145.669 85.479805) (end 145.669 84.8755) (width 0.25) (layer "F.Cu") (net 9))
-  (segment (start 151.8125 99.765195) (end 151.8125 85.93125) (width 0.25) (layer "F.Cu") (net 9))
-  (segment (start 151.8125 85.93125) (end 151.60625 85.725) (width 0.25) (layer "F.Cu") (net 9))
+  (segment (start 151.411053 85.944006) (end 146.133201 85.944006) (width 0.25) (layer "F.Cu") (net 9))
+  (segment (start 151.8125 86.51875) (end 151.8125 86.345453) (width 0.25) (layer "F.Cu") (net 9))
   (segment (start 145.669 85.479805) (end 145.669 84.987) (width 0.25) (layer "F.Cu") (net 9))
   (segment (start 149.495497 102.108) (end 149.495497 102.082198) (width 0.25) (layer "F.Cu") (net 9))
   (segment (start 149.495497 102.082198) (end 151.8125 99.765195) (width 0.25) (layer "F.Cu") (net 9))
-  (segment (start 151.60625 85.725) (end 145.914195 85.725) (width 0.25) (layer "F.Cu") (net 9))
   (via (at 243.459 57.15) (size 0.8) (drill 0.4) (layers "F.Cu" "B.Cu") (net 9))
   (via (at 110.109 57.15) (size 0.8) (drill 0.4) (layers "F.Cu" "B.Cu") (net 9))
@@
   (segment (start 149.479 102.124497) (end 149.479 105.877) (width 0.25) (layer "B.Cu") (net 9))
   (segment (start 149.495497 102.108) (end 149.479 102.124497) (width 0.25) (layer "B.Cu") (net 9))
+  (segment (start 147.189272 84.974626) (end 151.649626 84.974626) (width 0.25) (layer "F.Cu") (net 10))
+  (segment (start 151.649626 84.974626) (end 152.2625 85.5875) (width 0.25) (layer "F.Cu") (net 10))
   (segment (start 152.2625 100.3405) (end 150.495 102.108) (width 0.25) (layer "F.Cu") (net 10))
   (segment (start 147.193 84.836) (end 147.28825 84.93125) (width 0.25) (layer "F.Cu") (net 10))
-  (segment (start 147.28825 84.93125) (end 151.60625 84.93125) (width 0.25) (layer "F.Cu") (net 10))
   (segment (start 152.2625 85.5875) (end 152.2625 100.3405) (width 0.25) (layer "F.Cu") (net 10))
-  (segment (start 151.60625 84.93125) (end 152.2625 85.5875) (width 0.25) (layer "F.Cu") (net 10))
-  (via (at 147.193 84.836) (size 0.8) (drill 0.4) (layers "F.Cu" "B.Cu") (net 10))
   (via (at 55.372 76.2) (size 0.8) (drill 0.4) (layers "F.Cu" "B.Cu") (net 10))
   (via (at 191.135 76.2) (size 0.8) (drill 0.4) (layers "F.Cu" "B.Cu") (net 10))
   (via (at 133.985 76.2) (size 0.8) (drill 0.4) (layers "F.Cu" "B.Cu") (net 10))
+  (via (at 147.189272 84.974626) (size 0.8) (drill 0.4) (layers "F.Cu" "B.Cu") (net 10))
   (via (at 76.708 76.2) (size 0.8) (drill 0.4) (layers "F.Cu" "B.Cu") (net 10))
   (via (at 153.035 76.2) (size 0.8) (drill 0.4) (layers "F.Cu" "B.Cu") (net 10))
@@
   (arc (start 49.040744 83.848909) (mid 48.885881 83.617141) (end 48.8315 83.34375) (width 0.5) (layer "In1.Cu") (net 10))
   (arc (start 128.016 82.55) (mid 128.086017 82.198002) (end 128.285408 81.899593) (width 0.5) (layer "In1.Cu") (net 10))
+  (segment (start 147.189272 82.045728) (end 153.035 76.2) (width 0.25) (layer "B.Cu") (net 10))
+  (segment (start 147.189272 82.045728) (end 147.189272 84.974626) (width 0.25) (layer "B.Cu") (net 10))
   (segment (start 150.495 102.108) (end 150.495 105.877) (width 0.25) (layer "B.Cu") (net 10))
-  (segment (start 147.193 84.836) (end 147.193 82.042) (width 0.25) (layer "B.Cu") (net 10))
-  (segment (start 147.193 82.042) (end 153.035 76.2) (width 0.25) (layer "B.Cu") (net 10))
   (segment (start 142.592312 119.390501) (end 146.332687 119.390501) (width 0.25) (layer "B.Cu") (net 11))
   (segment (start 142.592312 119.390501) (end 142.592312 119.604972) (width 0.25) (layer "B.Cu") (net 11))
@@
   (arc (start 233.311682 73.181681) (mid 233.020315 72.74562) (end 232.918 72.23125) (width 0.5) (layer "In2.Cu") (net 23))
   (arc (start 232.918 62.755664) (mid 232.827233 62.299347) (end 232.56875 61.9125) (width 0.5) (layer "In2.Cu") (net 23))
+  (segment (start 228.6 102.11) (end 228.6 103.668888) (width 0.25) (layer "B.Cu") (net 23))
   (segment (start 224.857634 103.817) (end 228.451888 103.817) (width 0.25) (layer "B.Cu") (net 23))
   (segment (start 211.335121 105.6767) (end 212.020921 106.3625) (width 0.25) (layer "B.Cu") (net 23))
-  (segment (start 241.095 95.25) (end 234.362 101.983) (width 0.25) (layer "B.Cu") (net 23))
+  (segment (start 234.235 102.11) (end 241.095 95.25) (width 0.25) (layer "B.Cu") (net 23))
+  (segment (start 228.6 102.11) (end 234.235 102.11) (width 0.25) (layer "B.Cu") (net 23))
   (segment (start 222.312134 106.3625) (end 224.857634 103.817) (width 0.25) (layer "B.Cu") (net 23))
   (segment (start 212.020921 106.3625) (end 222.312134 106.3625) (width 0.25) (layer "B.Cu") (net 23))
-  (segment (start 228.6 103.668888) (end 228.6 101.983) (width 0.25) (layer "B.Cu") (net 23))
-  (segment (start 234.362 101.983) (end 228.6 101.983) (width 0.25) (layer "B.Cu") (net 23))
   (segment (start 208.55559 105.6767) (end 211.335121 105.6767) (width 0.25) (layer "B.Cu") (net 23))
   (segment (start 228.451888 103.817) (end 228.6 103.668888) (width 0.25) (layer "B.Cu") (net 23))
@@
   (via (at 166.878 114.3) (size 0.8) (drill 0.4) (layers "F.Cu" "B.Cu") (net 25))
   (via (at 133.555 114.3) (size 0.8) (drill 0.4) (layers "F.Cu" "B.Cu") (net 25))
-  (via (at 91.948 119.761) (size 0.8) (drill 0.4) (layers "F.Cu" "B.Cu") (net 25))
   (via (at 83.55 114.3) (size 0.8) (drill 0.4) (layers "F.Cu" "B.Cu") (net 25))
   (segment (start 173.13275 120.55475) (end 173.13528 120.55728) (width 0.5) (layer "In1.Cu") (net 25))
