File: matrix.kicad_sch (KiCad schematic)
At the start: 37 parts, among them SW1 EC_SW, SW10 EC_SW, SW11 EC_SW, SW12 EC_SW, SW13 EC_SW, SW14 EC_SW, SW15 EC_SW, SW16 EC_SW, SW17 EC_SW, SW18 EC_SW, SW19 EC_SW, SW2 EC_SW, SW20 EC_SW, SW21 EC_SW, SW22 EC_SW, SW23 EC_SW, SW24 EC_SW, SW25 EC_SW, SW26 EC_SW, SW27 EC_SW, SW28 EC_SW, SW29 EC_SW, SW3 EC_SW, SW30 EC_SW, SW31 EC_SW, SW32 EC_SW, SW33 EC_SW, SW34 EC_SW, SW35 EC_SW, SW36 EC_SW, SW37 EC_SW, SW4 EC_SW, SW5 EC_SW, SW6 EC_SW, SW7 EC_SW, SW8 EC_SW, SW9 EC_SW

Commit message: small schematic error fixed
Connections:
- net GND: now also SW11.3 (SG)
Changed lines of the file:
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@@
   (junction (at 227.33 168.91) (diameter 0) (color 0 0 0 0)
   )
+  (junction (at 336.55 109.855) (diameter 0) (color 0 0 0 0)
+  )
   (junction (at 125.73 168.91) (diameter 0) (color 0 0 0 0)
   )
@@
     (stroke (width 0) (type default))
   )
-  (wire (pts (xy 344.17 95.25) (xy 344.17 104.648))
+  (wire (pts (xy 344.17 95.25) (xy 344.17 104.775))
     (stroke (width 0) (type default))
   )
@@
     (stroke (width 0) (type default))
   )
-  (wire (pts (xy 311.15 109.855) (xy 349.25 109.855))
+  (wire (pts (xy 311.15 109.855) (xy 336.55 109.855))
     (stroke (width 0) (type default))
   )
@@
     (stroke (width 0) (type default))
   )
+  (wire (pts (xy 336.55 109.855) (xy 349.25 109.855))
+    (stroke (width 0) (type default))
+  )
   (wire (pts (xy 227.33 130.81) (xy 252.73 130.81))
     (stroke (width 0) (type default))
@@
     (stroke (width 0) (type default))
   )
+  (wire (pts (xy 328.93 104.775) (xy 328.93 111.125))
+    (stroke (width 0) (type default))
+  )
   (wire (pts (xy 100.33 130.81) (xy 125.73 130.81))
     (stroke (width 0) (type default))
@@
   )
   (wire (pts (xy 158.75 167.005) (xy 184.15 167.005))
-    (stroke (width 0) (type default))
-  )
-  (wire (pts (xy 328.93 104.648) (xy 328.93 111.125))
     (stroke (width 0) (type default))
   )
@@
     )
   )
-  (symbol (lib_id "cipulot_parts:EC_SW") (at 336.55 104.648 0) (unit 1)
-    (in_bom yes) (on_board yes) (dnp no) (fields_autoplaced)
-    (property "Reference" "SW11" (at 336.55 97.663 0)
-      (effects (font (size 1.27 1.27)))
-    )
-    (property "Value" "EC_SW" (at 336.55 100.203 0)
-      (effects (font (size 1.27 1.27)))
-    )
-    (property "Footprint" "cipulot_parts:ecs_pad_1U_no_ring" (at 336.55 104.648 0)
-      (effects (font (size 1.27 1.27)) hide)
-    )
-    (property "Datasheet" "" (at 336.55 104.648 0)
-      (effects (font (size 1.27 1.27)))
-    )
+  (symbol (lib_id "cipulot_parts:EC_SW") (at 336.55 104.775 0) (unit 1)
+    (in_bom yes) (on_board yes) (dnp no) (fields_autoplaced)
+    (property "Reference" "SW11" (at 336.55 97.79 0)
+      (effects (font (size 1.27 1.27)))
+    )
+    (property "Value" "EC_SW" (at 336.55 100.33 0)
+      (effects (font (size 1.27 1.27)))
+    )
+    (property "Footprint" "cipulot_parts:ecs_pad_1U_no_ring" (at 336.55 104.775 0)
+      (effects (font (size 1.27 1.27)) hide)
+    )
+    (property "Datasheet" "" (at 336.55 104.775 0)
+      (effects (font (size 1.27 1.27)))
+    )
