File: travaulta prototype.kicad_pcb (KiCad board)
At the start: 4 copper layers, 209.7 x 76.4 mm, 106 parts, among them SW1 EC_SW, SW10 EC_SW, SW11 EC_SW, SW12 EC_SW, SW13 EC_SW, SW14 EC_SW, SW15 EC_SW, SW16 EC_SW, SW17 EC_SW, SW18 EC_SW, SW19 EC_SW, SW2 EC_SW, SW20 EC_SW, SW21 EC_SW, SW22 EC_SW, SW23 EC_SW, SW24 EC_SW, SW25 EC_SW, SW26 EC_SW, SW27 EC_SW, SW28 EC_SW, SW29 EC_SW, SW3 EC_SW, SW30 EC_SW, SW31 EC_SW, SW32 EC_SW, SW33 EC_SW, SW34 EC_SW, SW35 EC_SW, SW36 EC_SW, SW37 EC_SW, SW38 BOOT0, SW4 EC_SW, SW5 EC_SW, SW6 EC_SW, SW7 EC_SW, SW8 EC_SW, SW9 EC_SW, U1 STM32F401CBUx, U2 XC6206PxxxMR, U3 74HC4051, U4 74HC4051, U5 OPA350, Y1 8 MHz

Commit message: fresh gerbers
deleted old plate gerbers, need new export
Parts:
- moved H16 0.79 mm to (175.4, 114.3)
- moved H15 0.79 mm to (123.0, 114.3)
- moved H9 0.79 mm to (70.6, 95.2)
- moved H13 0.79 mm to (232.6, 95.2)
Other:
- board text added: "reset"
Changed lines of the file:
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@@
   )
   (footprint "cipulot_parts:HOLE_M2" (layer "F.Cu")
-    (at 71.4375 95.25)
+    (at 70.64375 95.25)
     (property "Sheetfile" "mounting holes.kicad_sch")
     (property "Sheetname" "mounting holes")
@@
   )
   (footprint "cipulot_parts:HOLE_M2" (layer "F.Cu")
-    (at 231.775 95.25)
+    (at 232.56875 95.25)
     (property "Sheetfile" "mounting holes.kicad_sch")
     (property "Sheetname" "mounting holes")
@@
   )
   (footprint "cipulot_parts:HOLE_M2" (layer "F.Cu")
-    (at 122.2375 114.3)
+    (at 123.03125 114.3)
     (property "Sheetfile" "mounting holes.kicad_sch")
     (property "Sheetname" "mounting holes")
@@
   )
   (footprint "cipulot_parts:HOLE_M2" (layer "F.Cu")
-    (at 176.2125 114.3)
+    (at 175.41875 114.3)
     (property "Sheetfile" "mounting holes.kicad_sch")
     (property "Sheetname" "mounting holes")
@@
     (effects (font (size 0.8 0.8) (thickness 0.15)) (justify mirror))
   )
+  (gr_text "reset" (at 182.458831 118.400533) (layer "B.SilkS")
+    (effects (font (size 0.8 0.8) (thickness 0.15)) (justify left bottom mirror))
+  )
   (segment (start 84.188822 57.277) (end 84.198075 57.286253) (width 0.25) (layer "F.Cu") (net 1))

Commit message: pcb clean up, fresh gerbers
Routing:
- net COL9: track 91.0 -> 85.8 mm
- net AMUX_SEL_1: track 153.5 -> 149.5 mm
- net VBAT: track 319.6 -> 318.1 mm
- net APLEX_OUT_PIN_0: track 141.9 -> 140.6 mm
- net ADC: track 12.5 -> 11.5 mm
- net ROW3: track 222.5 -> 221.9 mm
