File: Project/travaulta.kicad_sch (KiCad schematic)
At the start: 26 parts, among them SW38 BOOT0, U1 STM32F401CBUx, U2 XC6206PxxxMR, Y1 8 MHz

Commit message: project cleanup
Parts:
- SW38: footprint Button_Switch_SMD:SW_Push_SPST_NO_Alps_SKRK -> Connector_PinHeader_2.54mm:PinHeader_1x02_P2.54mm_Vertical
