File: Project/travaulta.kicad_pcb (KiCad board)
At the start: 4 copper layers, 209.7 x 76.4 mm, 106 parts, among them SW1 EC_SW, SW10 EC_SW, SW11 EC_SW, SW12 EC_SW, SW13 EC_SW, SW14 EC_SW, SW15 EC_SW, SW16 EC_SW, SW17 EC_SW, SW18 EC_SW, SW19 EC_SW, SW2 EC_SW, SW20 EC_SW, SW21 EC_SW, SW22 EC_SW, SW23 EC_SW, SW24 EC_SW, SW25 EC_SW, SW26 EC_SW, SW27 EC_SW, SW28 EC_SW, SW29 EC_SW, SW3 EC_SW, SW30 EC_SW, SW31 EC_SW, SW32 EC_SW, SW33 EC_SW, SW34 EC_SW, SW35 EC_SW, SW36 EC_SW, SW37 EC_SW, SW38 BOOT0, SW4 EC_SW, SW5 EC_SW, SW6 EC_SW, SW7 EC_SW, SW8 EC_SW, SW9 EC_SW, U1 STM32F401CBUx, U2 XC6206PxxxMR, U3 74HC4051, U4 74HC4051, U5 OPA350, Y1 8 MHz

Commit message: project cleanup
Parts:
- SW38: footprint Button_Switch_SMD:SW_Push_SPST_NO_Alps_SKRK -> Connector_PinHeader_2.54mm:PinHeader_1x02_P2.54mm_Vertical
- moved R21 6.90 mm to (146.8, 119.4), turned to 0 degrees
- moved JP1 6.69 mm to (144.5, 120.7), turned to 180 degrees
- moved R16 5.78 mm to (234.2, 99.9), turned to -90 degrees
- moved R13 4.18 mm to (75.8, 107.2), turned to 180 degrees
- moved R23 2.61 mm to (142.1, 119.4)
- moved C14 2.22 mm to (140.7, 112.7)
- moved U5 2.15 mm to (144.4, 116.2)
- moved C12 1.84 mm to (203.1, 104.5)
- moved U3 1.77 mm to (205.6, 108.0)
- moved U4 1.77 mm to (92.9, 108.0)
- moved C13 1.75 mm to (88.9, 104.5), turned to 180 degrees
- moved R15 1.59 mm to (69.1, 100.0)
- moved SW38 1.27 mm to (181.0, 113.0), turned to 180 degrees
- moved R14 1.11 mm to (208.5, 112.1)
- moved H16 0.79 mm to (175.4, 114.3)
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Routing:
- net VBAT: track 296.4 -> 318.1 mm, vias 10 -> 9
- net ROW2: track 323.2 -> 308.5 mm
- net ROW0: track 373.4 -> 360.0 mm
- net ROW1: track 348.8 -> 335.6 mm
- net AMUX_SEL_0: track 155.1 -> 147.3 mm
- net APLEX_EN_PIN_1: track 73.7 -> 78.0 mm, vias 4 -> 2
- net COL1: track 87.1 -> 91.3 mm
- net AMUX_SEL_2: track 152.7 -> 148.7 mm
- net Net-(JP1-B): track 5.06 -> 8.98 mm
- net COL0: track 77.8 -> 81.4 mm
- net COL3: track 111.4 -> 115.0 mm
- net ADC: track 14.9 -> 11.5 mm
- net COL5: track 125.9 -> 128.8 mm
- net GND: track 40.4 -> 37.7 mm, vias 274 -> 326
- net APLEX_OUT_PIN_0: track 138.0 -> 140.6 mm, vias 5 -> 6
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Other:
- board text added: "by Calvin#0563 for projectcain#5265's vault35 Prototype"
- board text added: "reset"
- board text removed: "by Calvin#0563 for projectcain#5265's vault35"

Commit message: silkscreen labelling changed for GB
Other:
- board text added: "by Calvin0563 for mechvault's vault35"
- board text removed: "by Calvin#0563 for projectcain#5265's vault35 Prototype"
Changed lines of the file:
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@@
     (effects (font (size 1 1) (thickness 0.15)))
   )
-  (gr_text "by Calvin#0563\nfor projectcain#5265's vault35\nPrototype" (at 246.85625 76.2 270) (layer "B.SilkS")
-    (effects (font (size 0.8 0.8) (thickness 0.15)) (justify mirror))
+  (gr_text "by Calvin0563\nfor mechvault's vault35\n" (at 246.85625 76.2 270) (layer "B.SilkS")
+    (effects (font (size 1 1) (thickness 0.15)) (justify mirror))
   )
-  (gr_text "reset" (at 182.458831 118.400533) (layer "B.SilkS")
-    (effects (font (size 0.8 0.8) (thickness 0.15)) (justify left bottom mirror))
+  (gr_text "reset" (at 180.975 118.26875) (layer "B.SilkS")
+    (effects (font (size 1 1) (thickness 0.15)) (justify mirror))
   )
   (segment (start 84.188822 57.277) (end 84.198075 57.286253) (width 0.25) (layer "F.Cu") (net 1))
