File: Project/plates/travaulta plate topre.kicad_pcb (KiCad board)
At the start: 2 copper layers, 210.7 x 77.4 mm, 55 parts

Commit message: fresh set of production files
Other:
- board text added: "OEM plate"
- board text removed: "Topre Plate"
Changed lines of the file:
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@@
     (effects (font (size 1 1) (thickness 0.15)))
   )
-  (gr_text "Topre Plate" (at 247.65 76.2 270) (layer "F.SilkS")
-    (effects (font (size 0.8 0.8) (thickness 0.15)))
+  (gr_text "OEM plate" (at 247.65 76.2 270) (layer "F.SilkS")
+    (effects (font (size 1 1) (thickness 0.15)))
   )
   (gr_text "SW1" (at 201.6125 92.75) (layer "F.Fab")
