File: Project/plates/travaulta plate topre.kicad_pcb (KiCad board)
At the start: 2 copper layers, 210.7 x 77.4 mm, 55 parts

Commit message: plate files updated, new production files
Parts:
- removed ? (x16): , 
- removed H5: MountingHole, cipulot_parts:HOLE_M2
Changed lines of the file:
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@@
       (sketchpadsonfab false)
       (subtractmaskfromsilk false)
-      (outputformat 3)
+      (outputformat 1)
       (mirror false)
       (drillshape 0)
       (scaleselection 1)
-      (outputdirectory "production/plates/dxf")
+      (outputdirectory "production/plates/")
     )
   )
@@
     )
   )
-  (footprint "cipulot_parts:HOLE_M2" (layer "F.Cu")
-    (at 115.8875 95.25)
-    (property "Sheetfile" "mounting holes.kicad_sch")
-    (property "Sheetname" "mounting holes")
-    (attr through_hole board_only)
-    (fp_text reference "H5" (at 0 -2) (layer "F.SilkS") hide
-        (effects (font (size 0.29972 0.29972) (thickness 0.07493)))
-    )
-    (fp_text value "MountingHole" (at 0 2.2352) (layer "F.SilkS") hide
-        (effects (font (size 0.29972 0.29972) (thickness 0.0762)))
-    )
-    (pad "" np_thru_hole circle (at 0 0) (size 2.2 2.2) (drill 2.2) (layers "*.Cu" "*.Mask" "F.SilkS")
-      (clearance 0.5))
-  )
   (footprint "cipulot_parts:ecs_plate_cut_1U" (layer "F.Cu")
     (at 220.6625 95.25)
@@
     )
   )
-  (footprint "" (layer "F.Cu")
-    (at 175.41875 114.3)
-    (attr through_hole board_only)
-    (fp_text reference "" (at 0 0) (layer "F.SilkS")
-        (effects (font (size 1.27 1.27) (thickness 0.15)))
-    )
-    (fp_text value "" (at 0 0) (layer "F.SilkS")
-        (effects (font (size 1.27 1.27) (thickness 0.15)))
-    )
-    (pad "" np_thru_hole circle (at 0 0) (size 2.2 2.2) (drill 2.2) (layers "*.Cu" "*.Mask" "F.SilkS")
-      (clearance 0.5))
-  )
   (footprint "cipulot_parts:ecs_plate_cut_1U" (layer "F.Cu")
     (at 201.6125 95.25)
@@
     )
   )
-  (footprint "" (layer "F.Cu")
-    (at 70.64375 95.25)
-    (attr through_hole board_only)
-    (fp_text reference "" (at 0 0) (layer "F.SilkS")
-        (effects (font (size 1.27 1.27) (thickness 0.15)))
-    )
-    (fp_text value "" (at 0 0) (layer "F.SilkS")
-        (effects (font (size 1.27 1.27) (thickness 0.15)))
-    )
-    (pad "" np_thru_hole circle (at 0 0) (size 2.2 2.2) (drill 2.2) (layers "*.Cu" "*.Mask" "F.SilkS")
-      (clearance 0.5))
-  )
-  (footprint "" (layer "F.Cu")
-    (at 92.075 114.3)
-    (attr through_hole board_only)
-    (fp_text reference "" (at 0 0) (layer "F.SilkS")
-        (effects (font (size 1.27 1.27) (thickness 0.15)))
-    )
-    (fp_text value "" (at 0 0) (layer "F.SilkS")
-        (effects (font (size 1.27 1.27) (thickness 0.15)))
-    )
-    (pad "" np_thru_hole circle (at 0 0) (size 2.2 2.2) (drill 2.2) (layers "*.Cu" "*.Mask" "F.SilkS")
-      (clearance 0.5))
-  )
-  (footprint "" (layer "F.Cu")
-    (at 206.375 114.3)
-    (attr through_hole board_only)
-    (fp_text reference "" (at 0 0) (layer "F.SilkS")
-        (effects (font (size 1.27 1.27) (thickness 0.15)))
-    )
-    (fp_text value "" (at 0 0) (layer "F.SilkS")
-        (effects (font (size 1.27 1.27) (thickness 0.15)))
-    )
-    (pad "" np_thru_hole circle (at 0 0) (size 2.2 2.2) (drill 2.2) (layers "*.Cu" "*.Mask" "F.SilkS")
-      (clearance 0.5))
-  )
   (footprint "cipulot_parts:ecs_plate_cut_1U" (layer "F.Cu")
     (at 168.275 57.15)
@@
     )
   )
-  (footprint "" (layer "F.Cu")
-    (at 177.8 57.15)
-    (attr through_hole board_only)
-    (fp_text reference "" (at 0 0) (layer "F.SilkS")
-        (effects (font (size 1.27 1.27) (thickness 0.15)))
-    )
-    (fp_text value "" (at 0 0) (layer "F.SilkS")
-        (effects (font (size 1.27 1.27) (thickness 0.15)))
-    )
-    (pad "" np_thru_hole circle (at 0 0) (size 2.2 2.2) (drill 2.2) (layers "*.Cu" "*.Mask" "F.SilkS")
-      (clearance 0.5))
-  )
   (footprint "cipulot_parts:ecs_plate_cut_1U" (layer "F.Cu")
     (at 111.125 57.15)
@@
     )
   )
-  (footprint "" (layer "F.Cu")
-    (at 123.03125 114.3)
-    (attr through_hole board_only)
-    (fp_text reference "" (at 0 0) (layer "F.SilkS")
-        (effects (font (size 1.27 1.27) (thickness 0.15)))
-    )
-    (fp_text value "" (at 0 0) (layer "F.SilkS")
-        (effects (font (size 1.27 1.27) (thickness 0.15)))
-    )
-    (pad "" np_thru_hole circle (at 0 0) (size 2.2 2.2) (drill 2.2) (layers "*.Cu" "*.Mask" "F.SilkS")
-      (clearance 0.5))
-  )
   (footprint "cipulot_parts:ecs_plate_cut_1U" (layer "F.Cu")
     (at 182.5625 95.25)
@@
       (rotate (xyz 0 0 0))
     )
-  )
-  (footprint "" (layer "F.Cu")
-    (at 192.0875 95.25)
-    (attr through_hole board_only)
-    (fp_text reference "" (at 0 0) (layer "F.SilkS")
-        (effects (font (size 1.27 1.27) (thickness 0.15)))
-    )
-    (fp_text value "" (at 0 0) (layer "F.SilkS")
-        (effects (font (size 1.27 1.27) (thickness 0.15)))
-    )
-    (pad "" np_thru_hole circle (at 0 0) (size 2.2 2.2) (drill 2.2) (layers "*.Cu" "*.Mask" "F.SilkS")
-      (clearance 0.5))
-  )
-  (footprint "" (layer "F.Cu")
-    (at 120.65 57.15)
-    (attr through_hole board_only)
-    (fp_text reference "" (at 0 0) (layer "F.SilkS")
-        (effects (font (size 1.27 1.27) (thickness 0.15)))
-    )
-    (fp_text value "" (at 0 0) (layer "F.SilkS")
-        (effects (font (size 1.27 1.27) (thickness 0.15)))
-    )
-    (pad "" np_thru_hole circle (at 0 0) (size 2.2 2.2) (drill 2.2) (layers "*.Cu" "*.Mask" "F.SilkS")
-      (clearance 0.5))
   )
   (footprint "LOGO" (layer "F.Cu")
@@
       (stroke (width 0) (type solid)) (fill solid) (layer "F.SilkS"))
   )
-  (footprint "" (layer "F.Cu")
-    (at 220.6625 76.2)
-    (attr through_hole board_only)
-    (fp_text reference "" (at 0 0) (layer "F.SilkS")
-        (effects (font (size 1.27 1.27) (thickness 0.15)))
-    )
-    (fp_text value "" (at 0 0) (layer "F.SilkS")
-        (effects (font (size 1.27 1.27) (thickness 0.15)))
-    )
-    (pad "" np_thru_hole circle (at 0 0) (size 2.2 2.2) (drill 2.2) (layers "*.Cu" "*.Mask" "F.SilkS")
-      (clearance 0.5))
-  )
-  (footprint "" (layer "F.Cu")
-    (at 63.5 57.15)
-    (attr through_hole board_only)
-    (fp_text reference "" (at 0 0) (layer "F.SilkS")
-        (effects (font (size 1.27 1.27) (thickness 0.15)))
-    )
-    (fp_text value "" (at 0 0) (layer "F.SilkS")
-        (effects (font (size 1.27 1.27) (thickness 0.15)))
-    )
-    (pad "" np_thru_hole circle (at 0 0) (size 2.2 2.2) (drill 2.2) (layers "*.Cu" "*.Mask" "F.SilkS")
-      (clearance 0.5))
-  )
   (footprint "cipulot_parts:ecs_plate_cut_1U" (layer "F.Cu")
     (at 194.47 114.3)
@@
     )
   )
-  (footprint "" (layer "F.Cu")
-    (at 153.9875 95.25)
-    (attr through_hole board_only)
-    (fp_text reference "" (at 0 0) (layer "F.SilkS")
-        (effects (font (size 1.27 1.27) (thickness 0.15)))
-    )
-    (fp_text value "" (at 0 0) (layer "F.SilkS")
-        (effects (font (size 1.27 1.27) (thickness 0.15)))
-    )
-    (pad "" np_thru_hole circle (at 0 0) (size 2.2 2.2) (drill 2.2) (layers "*.Cu" "*.Mask" "F.SilkS")
-      (clearance 0.5))
-  )
-  (footprint "" (layer "F.Cu")
-    (at 87.3125 76.2)
-    (attr through_hole board_only)
-    (fp_text reference "" (at 0 0) (layer "Edge.Cuts")
-        (effects (font (size 1.27 1.27) (thickness 0.15)))
-    )
-    (fp_text value "" (at 0 0) (layer "Edge.Cuts")
-        (effects (font (size 1.27 1.27) (thickness 0.15)))
-    )
-    (pad "" np_thru_hole circle (at 0 0) (size 2.2 2.2) (drill 2.2) (layers "*.Cu" "*.Mask" "F.SilkS")
-      (clearance 0.5))
-  )
   (footprint "cipulot_parts:ecs_plate_cut_1U" (layer "F.Cu")
     (at 92.075 57.15)
@@
     )
   )
-  (footprint "" (layer "F.Cu")
-    (at 232.56875 95.25)
-    (attr through_hole board_only)
-    (fp_text reference "" (at 0 0) (layer "F.SilkS")
-        (effects (font (size 1.27 1.27) (thickness 0.15)))
-    )
-    (fp_text value "" (at 0 0) (layer "F.SilkS")
-        (effects (font (size 1.27 1.27) (thickness 0.15)))
-    )
-    (pad "" np_thru_hole circle (at 0 0) (size 2.2 2.2) (drill 2.2) (layers "*.Cu" "*.Mask" "F.SilkS")
-      (clearance 0.5))
-  )
   (footprint "cipulot_parts:ecs_plate_cut_1U" (layer "F.Cu")
     (at 242.095 95.25)
@@
     )
   )
-  (footprint "" (layer "F.Cu")
-    (at 234.95 57.15)
-    (attr through_hole board_only)
-    (fp_text reference "" (at 0 0) (layer "F.SilkS")
-        (effects (font (size 1.27 1.27) (thickness 0.15)))
-    )
-    (fp_text value "" (at 0 0) (layer "F.SilkS")
-        (effects (font (size 1.27 1.27) (thickness 0.15)))
-    )
-    (pad "" np_thru_hole circle (at 0 0) (size 2.2 2.2) (drill 2.2) (layers "*.Cu" "*.Mask" "F.SilkS")
-      (clearance 0.5))
-  )
   (footprint "cipulot_parts:ecs_plate_cut_1U" (layer "F.Cu")
     (at 106.3625 95.25)
@@
     )
   )
-  (footprint "" (layer "F.Cu")
-    (at 182.5625 76.2)
-    (attr through_hole board_only)
-    (fp_text reference "" (at 0 0) (layer "F.SilkS")
-        (effects (font (size 1.27 1.27) (thickness 0.15)))
-    )
-    (fp_text value "" (at 0 0) (layer "F.SilkS")
-        (effects (font (size 1.27 1.27) (thickness 0.15)))
-    )
-    (pad "" np_thru_hole circle (at 0 0) (size 2.2 2.2) (drill 2.2) (layers "*.Cu" "*.Mask" "F.SilkS")
-      (clearance 0.5))
-  )
-  (footprint "" (layer "F.Cu")
-    (at 125.4125 76.2)
-    (attr through_hole board_only)
-    (fp_text reference "" (at 0 0) (layer "F.SilkS")
-        (effects (font (size 1.27 1.27) (thickness 0.15)))
-    )
-    (fp_text value "" (at 0 0) (layer "F.SilkS")
-        (effects (font (size 1.27 1.27) (thickness 0.15)))
-    )
-    (pad "" np_thru_hole circle (at 0 0) (size 2.2 2.2) (drill 2.2) (layers "*.Cu" "*.Mask" "F.SilkS")
-      (clearance 0.5))
-  )
   (gr_circle (center 206.375 114.3) (end 207.525 114.3)
