File: Project/WKL/travaulta WKL.kicad_pcb (KiCad board)
At the start: 4 copper layers, 208.3 x 75.8 mm, 106 parts, among them SW1 EC_SW, SW10 EC_SW, SW11 EC_SW, SW12 EC_SW, SW13 EC_SW, SW14 EC_SW, SW15 EC_SW, SW16 EC_SW, SW17 EC_SW, SW18 EC_SW, SW19 EC_SW, SW2 EC_SW, SW20 EC_SW, SW21 EC_SW, SW22 EC_SW, SW23 EC_SW, SW24 EC_SW, SW25 EC_SW, SW26 EC_SW, SW27 EC_SW, SW28 EC_SW, SW29 EC_SW, SW3 EC_SW, SW30 EC_SW, SW31 EC_SW, SW32 EC_SW, SW33 EC_SW, SW34 EC_SW, SW35 EC_SW, SW36 EC_SW, SW37 EC_SW, SW38 BOOT0, SW4 EC_SW, SW5 EC_SW, SW6 EC_SW, SW7 EC_SW, SW8 EC_SW, SW9 EC_SW, U1 STM32F401CBUx, U2 XC6206PxxxMR, U3 74HC4051, U4 74HC4051, U5 OPA350, Y1 8 MHz

Commit message: wkl production files
Parts:
- moved G*** 2.38 mm to (250.8, 81.8)
Routing:
- net ROW2: track 314.3 -> 307.1 mm
- net GND: track 43.5 -> 46.9 mm, vias 333 -> 436
- net AMUX_SEL_2: track 107.9 -> 109.2 mm
- net AMUX_SEL_0: track 106.1 -> 107.5 mm
- net AMUX_SEL_1: track 109.3 -> 110.7 mm
- net COL10: track 114.5 -> 115.3 mm
- net COL8: track 93.9 -> 93.2 mm
- net ROW0: track 360.0 -> 359.3 mm
- net ROW1: track 335.6 -> 335.1 mm
- net COL3: vias 5 -> 4
