File: Project/travaulta HHKB/plates/travaulta plate naevies threaded.kicad_pcb (KiCad board)
At the start: 2 copper layers, 210.7 x 77.4 mm, 38 parts

Commit message: plate update
Other:
- outline, holes or cut-outs redrawn
