File: Project/travaulta HHKB/plates/travaulta plate topre fr4.kicad_pcb (KiCad board)
At the start: 2 copper layers, 210.7 x 77.4 mm, 38 parts

Commit message: plate update
Other:
- outline, holes or cut-outs redrawn
Changed lines of the file:
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@@
+		(layer "Edge.Cuts")
+	)
+	(gr_circle
+		(center 175.41875 114.3)
+		(end 176.56875 114.3)
+		(stroke
+			(width 0.2)
+			(type solid)
+		)
+		(fill none)
 		(layer "Edge.Cuts")
 	)
@@
 		(layer "Edge.Cuts")
 	)
-	(gr_circle
-		(center 175.41875 114.3)
-		(end 176.56875 114.3)
-		(stroke
-			(width 0.2)
-			(type solid)
-		)
-		(fill none)
-		(layer "Edge.Cuts")
-	)
 	(gr_arc
 		(start 226 106.974999)
@@
 		(layer "Edge.Cuts")
 	)
+	(gr_rect
+		(start 179.168161 111.215427)
+		(end 182.763392 117.358174)
+		(stroke
+			(width 0.1)
+			(type default)
+		)
+		(fill none)
+		(layer "Edge.Cuts")
+	)
 	(gr_circle
 		(center 182.5625 76.2)
@@
 		(net 1)
 		(net_name "GND")
-		(layers "F&B.Cu")
+		(layers "F.Cu" "B.Cu")
 		(hatch edge 0.508)
 		(connect_pads
